File: hw/ventilation_control/ventilation_control.kicad_pcb (KiCad board)
At the start: 2 copper layers, 70 x 90 mm, 183 parts, among them J1 SERVO1, J10 MOTOR2, J11 I2C2, J12 SPI1.2, J13 SPI1.6, J14 POWER, J15 USART3, J16 ADC, J17 SPI2, J18 SPI1.3, J19 SERVO3, J2 SERVO5, J20 SERVO7, J21 SPI1.7, J22 GPIO, J23 SPI1.4, J24 SPI1.8, J25 SERVO4, J26 SERVO8, J27 RS485_TERM, J28 RS-485, J3 MOTOR1, J4 PROG, J5 SPI1.1, J6 1WIRE, J7 SPI1.5, J8 SERVO2, J9 SERVO6, U1 TPS54331, U10 MAX485E, U11 INA180A1, U12 M24C01-WMN, U13 4051, U2 AMS1117-3.3, U3 LM358, U4 LM358, U5 LM358, U6 STM32G070CBT6, U7 LM358, U8 LM358, U9 74LS138, Y1 Crystal_GND23

Commit message: Final changes.
Parts:
- added C8: CP, Capacitor_THT:CP_Radial_D10.0mm_P5.00mm, B.Cu at (132.7, 40.7)
- R10: value R -> 10k
- R11: value R -> 1k8
- R9: value R -> 100R
Routing:
- net GND: vias 41 -> 224
Other:
- board text added: "+24V"
- board text added: "1WIRE"
- board text added: "24V"
- board text added: "3V3"
- board text added: "5V"
- board text added: "A"
- board text added: "ADC"
- board text added: "B"
- board text added: "CH1"
- board text added: "CH10"
- board text added: "CH2"
- board text added: "CH3"
- board text added: "CH4"
- board text added: "CH5"
- board text added: "CH6"
- board text added: "CH7"
- board text added: "CH8"
- board text added: "CH9"
- board text added: "GND"
- board text added: "GPIO"
- board text added: "I2C2"
- board text added: "IO0"
- board text added: "IO1"
- board text added: "IO2"
- board text added: "IO3"
- board text added: "MISO"
- board text added: "MOSI"
- board text added: "MOTORS"
- board text added: "OUTx"
- board text added: "POSx"
- board text added: "PROG"
- board text added: "RS-485"
- board text added: "RS-485 termination"
- board text added: "RX3"
- board text added: "SCK"
- board text added: "SCL2"
- board text added: "SDA2"
- board text added: "SERVO"
- board text added: "SPI SENSORS"
- board text added: "SPI1"
- board text added: "SPI2"
- board text added: "SS SCK2 MISO2 MOSI2 GND 3V3"
- board text added: "SWCLK"
- board text added: "SWDIO"
- board text added: "TX3"
- board text added: "USART3"
- board text added: "Ventilation controller v1 Jethro, 2022"
- board text added: "~{RST}"
- board text added: "~{SS}"
