File: hw/ventilation_control/ventilation_control.kicad_sch (KiCad schematic)
At the start: 184 parts, among them J1 SERVO1, J10 MOTOR2, J11 I2C2, J12 SPI1.2, J13 SPI1.6, J14 POWER, J15 USART3, J16 ADC, J17 SPI2, J18 SPI1.3, J19 SERVO3, J2 SERVO5, J20 SERVO7, J21 SPI1.7, J22 GPIO, J23 SPI1.4, J24 SPI1.8, J25 SERVO4, J26 SERVO8, J27 RS485_TERM, J28 RS-485, J3 MOTOR1, J4 PROG, J5 SPI1.1, J6 1WIRE, J7 SPI1.5, J8 SERVO2, J9 SERVO6, U1 TPS54331, U10 MAX485E, U11 INA180A1, U12 M24C01-WMN, U13 4051, U2 AMS1117-3.3, U3 LM358, U4 LM358, U5 LM358, U6 STM32G070CBT6, U7 LM358, U8 LM358, U9 74LS138, Y1 Crystal_GND23

Commit message: Final changes.
Parts:
- C11, C12, C13, C14, C15, C16, C18, C19, C20, C21, C22, C23, C24, C29, C30, C31, C32, C33, C34, C35, C36, C7: LCSC (none) -> C14663
- C2: LCSC (none) -> C29823
- C27, C28: value C -> 20pF; LCSC (none) -> C1648
- C3, C5: LCSC (none) -> C27920
- C4: LCSC (none) -> C21122
- C6: LCSC (none) -> C19702
- C8: value CP -> 330u; footprint (none) -> Capacitor_THT:CP_Radial_D10.0mm_P5.00mm
- C9: LCSC (none) -> C59461
- D4: LCSC (none) -> C133693
- F1: value Polyfuse -> SHV2920P500-30-AA; LCSC (none) -> C495350
- R1, R10: value R -> 10k; LCSC (none) -> C25804
- R11: value R -> 1k8; LCSC (none) -> C4177
- R12, R13, R14, R15, R16, R17, R38, R39, R40, R41, R52, R83: LCSC (none) -> C25819
- R18, R19, R20, R21, R22, R23, R46, R47, R48, R49, R65, R66, R67, R76, R78, R79, R80, R81, R82, R84: LCSC (none) -> C25804
- R2, R4: LCSC (none) -> C23162
- R24, R25, R26, R27, R28, R29, R50, R51, R53, R54, R57, R58, R59, R60, R61, R62, R63, R64: LCSC (none) -> C31850
- R30, R31, R32, R33, R34, R35, R36, R37, R42, R43, R44, R45, R56, R6, R68, R69, R7, R70, R71, R72, R73, R74, R75, R87: LCSC (none) -> C23138
- R5: value R -> 2k7; LCSC (none) -> C13167
- R55: value R -> 1M; LCSC (none) -> C22935
- R8: value R -> 1k; LCSC (none) -> C21190
- R85: LCSC (none) -> C22787
- R86, R88: LCSC (none) -> C25803
- R89: LCSC (none) -> C22790
- R9: value R -> 100R; LCSC (none) -> C22775
- U1: LCSC (none) -> C9865
- U13: value 4051 -> CD4051; LCSC (none) -> C21379
- U2: LCSC (none) -> C6186
- U3, U4, U5, U7, U8: LCSC (none) -> C7950
- U5: LCSC C7950 -> C7950
- U9: LCSC (none) -> C5602
- Y1: value Crystal_GND23 -> 16MHz
